Commit message: asdf

File: rsc/xarm6/xarm6_allegro_wrist_mounted_rotate copy.urdf (robot description, URDF)
Before this commit: robot xarm6, 29 links, 28 joints
Joints:
- joint gripper_base_joint: origin xyz=0 0.045 0.045 rpy=0 -1.57 -1.57 -> xyz=0 0.035 0.055 rpy=0 -1.57 -1.57
- joint index_tip: origin xyz=0 0 0.0267 rpy=0 0 0 -> xyz=0 0 0.0157 rpy=0 -1.570796 0
- joint middle_tip: origin xyz=0 0 0.0267 rpy=0 0 0 -> xyz=0 0 0.0157 rpy=0 -1.570796 0
- joint ring_tip: origin xyz=0 0 0.0267 rpy=0 0 0 -> xyz=0 0 0.0157 rpy=0 -1.570796 0
- joint thumb_tip: origin xyz=0 0 0.0423 rpy=0 0 0 -> xyz=0 0 0.0313 rpy=0 -1.570796 0
