Commit message: asdf

File: rsc/xarm6/xarm6.urdf (robot description, URDF)
Before this commit: robot xarm6, 29 links, 28 joints
Links:
- removed link index_base
- removed link index_distal
- removed link index_medial
- removed link index_proximal
- removed link index_tip
- removed link middle_base
- removed link middle_distal
- removed link middle_medial
- removed link middle_proximal
- removed link middle_tip
- removed link ring_base
- removed link ring_distal
- removed link ring_medial
- removed link ring_proximal
- removed link ring_tip
- removed link thumb_base
- removed link thumb_distal
- removed link thumb_medial
- removed link thumb_proximal
- removed link thumb_tip
Joints:
- removed joint index_base
- removed joint index_distal
- removed joint index_medial
- removed joint index_proximal
- removed joint index_tip
- removed joint middle_base
- removed joint middle_distal
- removed joint middle_medial
- removed joint middle_proximal
- removed joint middle_tip
- removed joint ring_base
- removed joint ring_distal
- removed joint ring_medial
- removed joint ring_proximal
- removed joint ring_tip
- removed joint thumb_base
- removed joint thumb_distal
- removed joint thumb_medial
- removed joint thumb_proximal
- removed joint thumb_tip
