Commit message: done with teleoperation in simulation fixed simulator and remove dependancy on input device and hands

File: rsc/robot/allegro/allegro.urdf (robot description, URDF)
Before this commit: robot xarm6, 28 links, 27 joints
Links:
- removed link allegro_root0
- removed link allegro_root1
- removed link allegro_root2
- removed link allegro_root3
- removed link allegro_root4
- removed link allegro_root5
- removed link world
- added link wrist
- link index_base: geometry collision mesh filename=allegro/meshes/primary_base.STL; visual mesh filename=allegro/meshes/primary_base.STL
- link index_distal: geometry collision mesh filename=allegro/meshes/primary_distal.STL; visual mesh filename=allegro/meshes/primary_distal.STL
- link index_medial: geometry collision mesh filename=allegro/meshes/primary_medial.STL; visual mesh filename=allegro/meshes/primary_medial.STL
- link index_proximal: geometry collision mesh filename=allegro/meshes/primary_proximal.STL; visual mesh filename=allegro/meshes/primary_proximal.STL
- link index_tip: geometry collision sphere radius=0.015; visual mesh filename=allegro/meshes/primary_tip.STL
- link middle_base: geometry collision mesh filename=allegro/meshes/primary_base.STL; visual mesh filename=allegro/meshes/primary_base.STL
- link middle_distal: geometry collision mesh filename=allegro/meshes/primary_distal.STL; visual mesh filename=allegro/meshes/primary_distal.STL
- link middle_medial: geometry collision mesh filename=allegro/meshes/primary_medial.STL; visual mesh filename=allegro/meshes/primary_medial.STL
- link middle_proximal: geometry collision mesh filename=allegro/meshes/primary_proximal.STL; visual mesh filename=allegro/meshes/primary_proximal.STL
- link middle_tip: geometry collision sphere radius=0.015; visual mesh filename=allegro/meshes/primary_tip.STL
- link palm_link: geometry collision mesh filename=allegro/meshes/palm_link.obj; visual mesh filename=allegro/meshes/palm_link.obj
- link ring_base: geometry collision mesh filename=allegro/meshes/primary_base.STL; visual mesh filename=allegro/meshes/primary_base.STL
- link ring_distal: geometry collision mesh filename=allegro/meshes/primary_distal.STL; visual mesh filename=allegro/meshes/primary_distal.STL
- link ring_medial: geometry collision mesh filename=allegro/meshes/primary_medial.STL; visual mesh filename=allegro/meshes/primary_medial.STL
- link ring_proximal: geometry collision mesh filename=allegro/meshes/primary_proximal.STL; visual mesh filename=allegro/meshes/primary_proximal.STL
- link ring_tip: geometry collision sphere radius=0.015; visual mesh filename=allegro/meshes/primary_tip.STL
- link thumb_base: geometry collision mesh filename=allegro/meshes/thumb_base.STL; visual mesh filename=allegro/meshes/thumb_base.STL
- link thumb_distal: geometry collision mesh filename=allegro/meshes/thumb_distal.STL; visual mesh filename=allegro/meshes/thumb_distal.STL
- link thumb_medial: geometry collision mesh filename=allegro/meshes/thumb_medial.STL; visual mesh filename=allegro/meshes/thumb_medial.STL
- link thumb_proximal: geometry collision mesh filename=allegro/meshes/thumb_proximal.STL; visual mesh filename=allegro/meshes/thumb_proximal.STL
- link thumb_tip: geometry collision sphere radius=0.0145; visual mesh filename=allegro/meshes/thumb_tip.STL
Joints:
- removed joint world_joint
- removed joint x_joint
- removed joint x_rotation_joint
- removed joint y_joint
- removed joint y_rotation_joint
- removed joint z_joint
- removed joint z_rotation_joint
- added joint palm_link: type fixed, parent wrist, child palm_link, origin xyz=0.0095 0 0.095 rpy=0 0 0

File: rsc/robot/xarm.urdf (robot description, URDF)
Before this commit: robot xarm6, 9 links, 8 joints
Links:
- removed link palm_link
- link link1: geometry collision mesh filename=xarm/meshes/link1.obj; visual mesh filename=xarm/meshes/link1.obj
- link link2: geometry collision mesh filename=xarm/meshes/link2.obj; visual mesh filename=xarm/meshes/link2.obj
- link link3: geometry collision mesh filename=xarm/meshes/link3.obj; visual mesh filename=xarm/meshes/link3.obj
- link link4: geometry collision mesh filename=xarm/meshes/link4.obj; visual mesh filename=xarm/meshes/link4.obj
- link link5: geometry collision mesh filename=xarm/meshes/link5.obj; visual mesh filename=xarm/meshes/link5.obj
- link link6: geometry collision mesh filename=xarm/meshes/link6.obj; visual mesh filename=xarm/meshes/link6.obj
- link link_base: geometry collision mesh filename=xarm/meshes/base.obj; visual mesh filename=xarm/meshes/base.obj
Joints:
- removed joint gripper_base_joint

File: rsc/robot/xarm_allegro.urdf (robot description, URDF)
Before this commit: robot xarm6, 29 links, 28 joints
Links:
- added link wrist
- link index_tip: geometry collision sphere radius=0.015; visual mesh filename=allegro/meshes/primary_tip.STL
- link middle_tip: geometry collision sphere radius=0.015; visual mesh filename=allegro/meshes/primary_tip.STL
- link ring_tip: geometry collision sphere radius=0.015; visual mesh filename=allegro/meshes/primary_tip.STL
- link thumb_tip: geometry collision sphere radius=0.0145; visual mesh filename=allegro/meshes/thumb_tip.STL
Joints:
- removed joint gripper_base_joint
- added joint arm_to_hand: type fixed, parent link6, child wrist, origin xyz=0.00000 0.00000 0.04500 rpy=0.00000 0.00000 -1.57080
- added joint palm_link: type fixed, parent wrist, child palm_link, origin xyz=0.0095 0 0.095 rpy=0 0 0
- joint index_tip: origin xyz=0 0 0.0157 rpy=0 -1.570796 0 -> xyz=0 0 0.0267 rpy=0 0 0
- joint middle_tip: origin xyz=0 0 0.0157 rpy=0 -1.570796 0 -> xyz=0 0 0.0267 rpy=0 0 0
- joint ring_tip: origin xyz=0 0 0.0157 rpy=0 -1.570796 0 -> xyz=0 0 0.0267 rpy=0 0 0
- joint thumb_tip: origin xyz=0 0 0.0313 rpy=0 -1.570796 0 -> xyz=0 0 0.0423 rpy=0 0 0
