Commit message: ㅁㄴㅇㄹ

File: rsc/robot/xarm_inspire copy.urdf (robot description, URDF)
Before this commit: robot combined_robot, 22 links, 21 joints
Joints:
- joint arm_to_hand: origin xyz=0.00000 0.00000 0.03500 rpy=3.14159 0.00000 0.78540 -> xyz=0.00000 0.00000 0.03500 rpy=3.14159 0.00000 0.00000
