Commit message: asdf

File: rsc/robot/inspire copy.urdf (robot description, URDF)
Before this commit: robot combined_robot, 22 links, 21 joints
Links:
- removed link link1
- removed link link2
- removed link link3
- removed link link4
- removed link link5
- removed link link6
- removed link link_base
- removed link world
Joints:
- removed joint arm_to_hand
- removed joint joint1
- removed joint joint2
- removed joint joint3
- removed joint joint4
- removed joint joint5
- removed joint joint6
- removed joint world_joint
