Commit message: asdf

File: rsc/robot/allegro_float.urdf (robot description, URDF)
Before this commit: robot allegro, 29 links, 28 joints
Links:
- link index_tip: geometry collision sphere radius=0.015; visual mesh filename=allegro/meshes/tip.STL
- link middle_tip: geometry collision sphere radius=0.015; visual mesh filename=allegro/meshes/tip.STL
- link ring_tip: geometry collision sphere radius=0.015; visual mesh filename=allegro/meshes/tip.STL
- link thumb_tip: geometry collision sphere radius=0.0145; visual mesh filename=allegro/meshes/tip.STL
Joints:
- joint index_tip: origin xyz=0 0 0.0267 rpy=0 0 0 -> xyz=0 0 0.0157 rpy=0 -1.570796 0
- joint middle_tip: origin xyz=0 0 0.0267 rpy=0 0 0 -> xyz=0 0 0.0157 rpy=0 -1.570796 0
- joint ring_tip: origin xyz=0 0 0.0267 rpy=0 0 0 -> xyz=0 0 0.0157 rpy=0 -1.570796 0
- joint thumb_tip: origin xyz=0 0 0.0423 rpy=0 0 0 -> xyz=0 0 0.0313 rpy=0 -1.570796 0

File: rsc/robot/xarm_allegro.urdf (robot description, URDF)
Before this commit: robot combined_robot, 30 links, 29 joints
Links:
- link index_tip: geometry collision sphere radius=0.015; visual mesh filename=allegro/meshes/tip.STL
- link middle_tip: geometry collision sphere radius=0.015; visual mesh filename=allegro/meshes/tip.STL
- link ring_tip: geometry collision sphere radius=0.015; visual mesh filename=allegro/meshes/tip.STL
- link thumb_tip: geometry collision sphere radius=0.0145; visual mesh filename=allegro/meshes/tip.STL
Joints:
- joint arm_to_hand: origin xyz=-0.0001435 0.00139 0.06019 rpy=0.00000 0.00000 -1.57080 -> xyz=0.001273 -0.00054 0.06132 rpy=-0.00526 0.012665 -1.5592912
- joint index_tip: origin xyz=0 0 0.0267 rpy=0 0 0 -> xyz=0 0 0.0157 rpy=0 -1.570796 0
- joint middle_tip: origin xyz=0 0 0.0267 rpy=0 0 0 -> xyz=0 0 0.0157 rpy=0 -1.570796 0
- joint ring_tip: origin xyz=0 0 0.0267 rpy=0 0 0 -> xyz=0 0 0.0157 rpy=0 -1.570796 0
- joint thumb_tip: origin xyz=0 0 0.0423 rpy=0 0 0 -> xyz=0 0 0.0313 rpy=0 -1.570796 0
