Commit message: adf

File: rsc/robot/xarm_allegro.urdf (robot description, URDF)
Before this commit: robot combined_robot, 30 links, 29 joints
Joints:
- removed joint palm_link
- added joint palm_joint: type fixed, parent wrist, child palm_link, origin xyz=0.0095 0 0.095 rpy=0 0 0

Commit message: Remove large model file

File: rsc/robot/xarm_allegro.urdf (robot description, URDF)
Before this commit: robot combined_robot, 30 links, 29 joints
Joints:
- joint arm_to_hand: origin xyz=0.00000 0.00000 0.04500 rpy=0.00000 0.00000 -1.57080 -> xyz=0.00000 0.00000 0.0500 rpy=0.00000 0.00000 -1.57080

Commit message: asdf

File: rsc/robot/xarm_allegro.urdf (robot description, URDF)
Before this commit: robot combined_robot, 30 links, 29 joints
Joints:
- joint arm_to_hand: origin xyz=0.00000 0.00000 0.0500 rpy=0.00000 0.00000 -1.57080 -> xyz=-0.0001435 0.00139 0.06019 rpy=0.00000 0.00000 -1.57080

Commit message: asdf

File: rsc/robot/xarm_allegro.urdf (robot description, URDF)
Before this commit: robot combined_robot, 30 links, 29 joints
Joints:
- joint arm_to_hand: origin xyz=0.001273 -0.00054 0.06132 rpy=-0.00526 0.012665 -1.5592912 -> xyz=0.001 0.0002 0.06016 rpy=0 0 -1.570796
