Commit message: a lot of stuffs

File: rsc/robot/inspire_left.urdf (robot description, URDF)
Before this commit: robot inspire_hand_left, 19 links, 18 joints
Links:
- removed link base
- removed link hand_base_link
- removed link index_intermediate
- removed link index_proximal
- removed link index_tip
- removed link middle_intermediate
- removed link middle_proximal
- removed link middle_tip
- removed link pinky_intermediate
- removed link pinky_proximal
- removed link pinky_tip
- removed link ring_intermediate
- removed link ring_proximal
- removed link ring_tip
- removed link thumb_distal
- removed link thumb_intermediate
- removed link thumb_proximal
- removed link thumb_proximal_base
- removed link thumb_tip
- added link base_link, mass 0.260034351097693; collision mesh filename=inspire/meshes_left/base_link.STL; visual mesh filename=inspire/meshes_left/base_link.STL
- added link left_index_1, mass 0.0071995003148682; collision mesh filename=inspire/meshes_left/left_index_1.STL; visual mesh filename=inspire/meshes_left/left_index_1.STL
- added link left_index_2, mass 0.00968688267109518; collision mesh filename=inspire/meshes_left/left_index_2.STL; visual mesh filename=inspire/meshes_left/left_index_2.STL
- added link left_little_1, mass 0.0071994553320001; collision mesh filename=inspire/meshes_left/left_little_1.STL; visual mesh filename=inspire/meshes_left/left_little_1.STL
- added link left_little_2, mass 0.00759267726265222; collision mesh filename=inspire/meshes_left/left_little_2.STL; visual mesh filename=inspire/meshes_left/left_little_2.STL
- added link left_middle_1, mass 0.00719950322487974; collision mesh filename=inspire/meshes_left/left_middle_1.STL; visual mesh filename=inspire/meshes_left/left_middle_1.STL
- added link left_middle_2, mass 0.0104611931926301; collision mesh filename=inspire/meshes_left/left_middle_2.STL; visual mesh filename=inspire/meshes_left/left_middle_2.STL
- added link left_ring_1, mass 0.00719949770218712; collision mesh filename=inspire/meshes_left/left_ring_1.STL; visual mesh filename=inspire/meshes_left/left_ring_1.STL
- added link left_ring_2, mass 0.00968685177133057; collision mesh filename=inspire/meshes_left/left_ring_2.STL; visual mesh filename=inspire/meshes_left/left_ring_2.STL
- added link left_thumb_1, mass 0.00115518743162309; collision mesh filename=inspire/meshes_left/left_thumb_1.STL; visual mesh filename=inspire/meshes_left/left_thumb_1.STL
- added link left_thumb_2, mass 0.016; collision mesh filename=inspire/meshes_left/left_thumb_2.STL; visual mesh filename=inspire/meshes_left/left_thumb_2.STL
- added link left_thumb_3, mass 0.012; collision mesh filename=inspire/meshes_left/left_thumb_3.STL; visual mesh filename=inspire/meshes_left/left_thumb_3.STL
- added link left_thumb_4, mass 0.01; collision mesh filename=inspire/meshes_left/left_thumb_4.STL; visual mesh filename=inspire/meshes_left/left_thumb_4.STL
- added link world
Joints:
- removed joint base_joint
- removed joint index_intermediate_joint
- removed joint index_proximal_joint
- removed joint index_tip_joint
- removed joint middle_intermediate_joint
- removed joint middle_proximal_joint
- removed joint middle_tip_joint
- removed joint pinky_intermediate_joint
- removed joint pinky_proximal_joint
- removed joint pinky_tip_joint
- removed joint ring_intermediate_joint
- removed joint ring_proximal_joint
- removed joint ring_tip_joint
- removed joint thumb_distal_joint
- removed joint thumb_intermediate_joint
- removed joint thumb_proximal_pitch_joint
- removed joint thumb_proximal_yaw_joint
- removed joint thumb_tip_joint
- added joint L_hand_base_joint: type fixed, parent world, child base_link, origin xyz=0.5 0.5 0.001 rpy=3.14  0 -1.57
- added joint left_index_1_joint: type revolute, parent base_link, child left_index_1, origin xyz=0.025387 -0.00056467 -0.15686 rpy=-1.6057 0 1.5708, axis 0 0 1, limit lower=0 upper=1.6 effort=10 velocity=1
- added joint left_index_2_joint: type revolute, parent left_index_1, child left_index_2, origin xyz=-0.0016312 0.032734 -0.00055 rpy=0 0 0, axis 0 0 1, limit lower=0 upper=3.14 effort=10 velocity=1, mimic joint=left_index_1_joint multiplier=1.05 offset=0
- added joint left_little_1_joint: type revolute, parent base_link, child left_little_1, origin xyz=-0.039144 -0.00056467 -0.15226 rpy=-1.4661 0 1.5708, axis 0 0 1, limit lower=0 upper=1.6 effort=10 velocity=1
- added joint left_little_2_joint: type revolute, parent left_little_1, child left_little_2, origin xyz=-0.005182 0.032363 -0.00055 rpy=0 0 0, axis 0 0 1, limit lower=0 upper=3.14 effort=10 velocity=1, mimic joint=left_little_1_joint multiplier=1.18 offset=0
- added joint left_middle_1_joint: type revolute, parent base_link, child left_middle_1, origin xyz=0.0037996 -0.00056467 -0.157 rpy=-1.5708 0 1.5708, axis 0 0 1, limit lower=0 upper=1.6 effort=1 velocity=1
- added joint left_middle_2_joint: type revolute, parent left_middle_1, child left_middle_2, origin xyz=-0.0028436 0.032651 -0.00055 rpy=0 0 0, axis 0 0 1, limit lower=0 upper=3.14 effort=10 velocity=1, mimic joint=left_middle_1_joint multiplier=1.05 offset=0
- added joint left_ring_1_joint: type revolute, parent base_link, child left_ring_1, origin xyz=-0.017813 -0.00056467 -0.15614 rpy=-1.5184 0 1.5708, axis 0 0 1, limit lower=0 upper=1.6 effort=10 velocity=1
- added joint left_ring_2_joint: type revolute, parent left_ring_1, child left_ring_2, origin xyz=-0.0031431 0.032624 -0.00055 rpy=0 0 0, axis 0 0 1, limit lower=0 upper=3.14 effort=10 velocity=1, mimic joint=left_ring_1_joint multiplier=1.05 offset=0
- added joint left_thumb_1_joint: type revolute, parent base_link, child left_thumb_1, origin xyz=0.0269 -0.02101 -0.07075 rpy=0 0 0, axis 0 0 -1, limit lower=0 upper=1.15 effort=10 velocity=1
- added joint left_thumb_2_joint: type revolute, parent left_thumb_1, child left_thumb_2, origin xyz=0.0063016 -0.011924 -0.00125 rpy=-1.5708 0 -0.34907, axis 0 0 1, limit lower=0 upper=0.55 effort=10 velocity=1
- added joint left_thumb_3_joint: type revolute, parent left_thumb_2, child left_thumb_3, origin xyz=0.026828 0.02583 0.00315 rpy=0 0 0, axis 0 0 1, limit lower=0 upper=3.14 effort=10 velocity=1, mimic joint=left_thumb_2_joint multiplier=0.60 offset=0
- added joint left_thumb_4_joint: type revolute, parent left_thumb_3, child left_thumb_4, origin xyz=0.027027 0.0069965 -0.00145 rpy=0 0 0, axis 0 0 1, limit lower=0 upper=3.14 effort=10 velocity=1, mimic joint=left_thumb_2_joint multiplier=0.8 offset=0
