Commit message: lefthand

File: rsc/robot/xarm_inspire_left_new.urdf (robot description, URDF)
Before this commit: robot combined_robot, 22 links, 21 joints
Joints:
- joint arm_to_hand: origin xyz=0.00000 0.00000 0.0380 rpy=3.14159 0.00000 0.00000 -> xyz=0.00450 0.00000 0.0350 rpy=3.11 0.00000 0.0000
- joint left_index_2_joint: mimic joint=left_index_1_joint multiplier=1.05 offset=0 -> joint=left_index_1_joint multiplier=0.67 offset=0.22
- joint left_little_2_joint: limit lower=0 upper=3.14 effort=10 velocity=1 -> lower=-0.04545 upper=1.56 effort=1 velocity=0.5; mimic joint=left_little_1_joint multiplier=1.18 offset=0 -> joint=left_little_1_joint multiplier=0.9889 offset=-0.03126
- joint left_middle_2_joint: mimic joint=left_middle_1_joint multiplier=1.05 offset=0 -> joint=left_middle_1_joint multiplier=0.88 offset=0.15
- joint left_thumb_3_joint: mimic joint=left_thumb_2_joint multiplier=0.60 offset=0 -> joint=left_thumb_2_joint multiplier=1.114 offset=0
- joint left_thumb_4_joint: mimic joint=left_thumb_2_joint multiplier=0.8 offset=0 -> joint=left_thumb_2_joint multiplier=0.62 offset=0
