Commit message: asdf

File: rsc/robot/xarm_inspire_left_new_floating.urdf (robot description, URDF)
Before this commit: robot combined_robot, 22 links, 21 joints
Links:
- added link arm_to_hand_pitch
- added link arm_to_hand_roll
- added link arm_to_hand_x
- added link arm_to_hand_y
- added link arm_to_hand_yaw
- added link arm_to_hand_z
Joints:
- removed joint arm_to_hand
- added joint arm_to_hand_pitch: type continuous, parent arm_to_hand_roll, child arm_to_hand_pitch, axis 0 1 0
- added joint arm_to_hand_roll: type continuous, parent arm_to_hand_z, child arm_to_hand_roll, axis 1 0 0
- added joint arm_to_hand_x: type prismatic, parent link6, child arm_to_hand_x, origin xyz=0 0 0.0350 rpy=3.141592 0 0, axis 1 0 0, limit lower=-0.05 upper=0.05 effort=1 velocity=1
- added joint arm_to_hand_y: type prismatic, parent arm_to_hand_x, child arm_to_hand_y, axis 0 1 0, limit lower=-0.05 upper=0.05 effort=1 velocity=1
- added joint arm_to_hand_yaw: type continuous, parent arm_to_hand_pitch, child wrist, axis 0 0 1
- added joint arm_to_hand_z: type prismatic, parent arm_to_hand_y, child arm_to_hand_z, axis 0 0 1, limit lower=-0.05 upper=0.05 effort=1 velocity=1
