Commit message: rlworld_demo

File: rsc/robot/xarm_inspire.urdf (robot description, URDF)
Before this commit: robot combined_robot, 22 links, 21 joints
Joints:
- joint arm_to_hand: origin xyz=0.00000 0.00000 0.03500 rpy=3.14159 0.00000 0.00000 -> xyz=0.00000 0.00000 0.0600 rpy=3.14159 0.00000 0.00000

Commit message: asdf

File: rsc/robot/xarm_inspire.urdf (robot description, URDF)
Before this commit: robot combined_robot, 22 links, 21 joints
Joints:
- joint arm_to_hand: origin xyz=0.00000 0.00000 0.0600 rpy=3.14159 0.00000 0.00000 -> xyz=0.00000 0.00000 0.0250 rpy=3.14159 0.00000 0.00000

Commit message: asdf[::2

File: rsc/robot/xarm_inspire.urdf (robot description, URDF)
Before this commit: robot combined_robot, 22 links, 21 joints
Joints:
- joint arm_to_hand: origin xyz=0.00000 0.00000 0.0250 rpy=3.14159 0.00000 0.00000 -> xyz=0.00000 0.00000 0.0350 rpy=3.14159 0.00000 0.00000

Commit message: asdf

File: rsc/robot/xarm_inspire.urdf (robot description, URDF)
Before this commit: robot combined_robot, 22 links, 21 joints
Joints:
- joint arm_to_hand: origin xyz=0.00000 0.00000 0.0350 rpy=3.14159 0.00000 0.00000 -> xyz=0.00000 0.00000 -0.03500 rpy=3.14159 0.00000 0.00000

Commit message: hand calibration

File: rsc/robot/xarm_inspire.urdf (robot description, URDF)
Before this commit: robot combined_robot, 22 links, 21 joints
Links:
- link base_link: geometry collision mesh filename=inspire/meshes_right/base_link.STL; visual mesh filename=inspire/meshes_right/base_link.STL
- link right_index_1: geometry collision mesh filename=inspire/meshes_right/right_index_1.STL; visual mesh filename=inspire/meshes_right/right_index_1.STL
- link right_index_2: geometry collision mesh filename=inspire/meshes_right/right_index_2.STL; visual mesh filename=inspire/meshes_right/right_index_2.STL
- link right_little_1: geometry collision mesh filename=inspire/meshes_right/right_little_1.STL; visual mesh filename=inspire/meshes_right/right_little_1.STL
- link right_little_2: geometry collision mesh filename=inspire/meshes_right/right_little_2.STL; visual mesh filename=inspire/meshes_right/right_little_2.STL
- link right_middle_1: geometry collision mesh filename=inspire/meshes_right/right_middle_1.STL; visual mesh filename=inspire/meshes_right/right_middle_1.STL
- link right_middle_2: geometry collision mesh filename=inspire/meshes_right/right_middle_2.STL; visual mesh filename=inspire/meshes_right/right_middle_2.STL
- link right_ring_1: geometry collision mesh filename=inspire/meshes_right/right_ring_1.STL; visual mesh filename=inspire/meshes_right/right_ring_1.STL
- link right_ring_2: geometry collision mesh filename=inspire/meshes_right/right_ring_2.STL; visual mesh filename=inspire/meshes_right/right_ring_2.STL
- link right_thumb_1: geometry collision mesh filename=inspire/meshes_right/right_thumb_1.STL; visual mesh filename=inspire/meshes_right/right_thumb_1.STL
- link right_thumb_2: geometry collision mesh filename=inspire/meshes_right/right_thumb_2.STL; visual mesh filename=inspire/meshes_right/right_thumb_2.STL
- link right_thumb_3: geometry collision mesh filename=inspire/meshes_right/right_thumb_3.STL; visual mesh filename=inspire/meshes_right/right_thumb_3.STL
- link right_thumb_4: geometry collision mesh filename=inspire/meshes_right/right_thumb_4.STL; visual mesh filename=inspire/meshes_right/right_thumb_4.STL
Joints:
- joint arm_to_hand: origin xyz=0.00000 0.00000 -0.03500 rpy=3.14159 0.00000 0.00000 -> xyz=0.00000 0.00000 0.03500 rpy=3.14159 0.00000 0.00000
