Commit message: feat(hri): add keyboard-driven xarm_f1 capture flow and URDF merge fallback
- add keyboard session controls for robot capture (`c/s/q`) and grasp result labeling (`y/n`)
- extend teleop loop with event-based start/stop/exit and selectable control policy
- save hand-side capture outputs under structured `capture/hri_taeyun/...` paths with C2R export
- add inspire_f1 right-hand URDF resolution and new merged `xarm_inspire_f1_right.urdf`
- update xacro include/arg syntax and add XML-based fallback merge when xacro execution fails
- improve robot projection/loading for `inspire_f1` datasets and missing hand timestamps
- add camera gain/exposure config for `system/paradex1/camera.json`

File: rsc/robot/robot_combined.urdf.xacro (robot description, xacro)
@@ -6,10 +6,10 @@
   <xacro:arg name="xyz" default="0 0 0"/>
   <xacro:arg name="rpy" default="0 0 0"/>
-  <xacro:include filename="$(arg arm_file)" />
-  <xacro:include filename="$(arg hand_file)" />
+  <xacro:include filename="${arm_file}" />
+  <xacro:include filename="${hand_file}" />
   <joint name="arm_to_hand" type="fixed">
-    <parent link="$(arg parent_link)"/>
-    <child link="$(arg child_link)"/>
-    <origin xyz="$(arg xyz)" rpy="$(arg rpy)"/>
+    <parent link="${parent_link}"/>
+    <child link="${child_link}"/>
+    <origin xyz="${xyz}" rpy="${rpy}"/>
   </joint>
 </robot>
