Commit message: visualization code updated

File: rsc/robot/xarm_inspire_f1_right.urdf (robot description, URDF)
Before this commit: robot combined_robot, 36 links, 35 joints
Joints:
- joint right_thumb_4_joint: mimic joint=right_thumb_3_joint multiplier=0.8962 offset=0 -> joint=right_thumb_2_joint multiplier=1.1608 offset=0

Commit message: dp 3cam

File: rsc/robot/xarm_inspire_f1_right.urdf (robot description, URDF)
Before this commit: robot combined_robot, 36 links, 35 joints
Links:
- link index_force_sensor: mass 0 -> 0.01
- link index_tip: mass 0 -> 0.01
- link little_force_sensor: mass 0 -> 0.01
- link little_tip: mass 0 -> 0.01
- link middle_force_sensor: mass 0 -> 0.01
- link middle_tip: mass 0 -> 0.01
- link ring_force_sensor: mass 0 -> 0.01
- link ring_tip: mass 0 -> 0.01
- link thumb_force_sensor: mass 0 -> 0.01
- link thumb_tip: mass 0 -> 0.01
