Commit message: ㅁㄴㅇㄹ

File: rsc/robot/xarm.urdf (robot description, URDF)
Before this commit: robot xarm6, 8 links, 7 joints
Joints:
- joint joint1: origin xyz=0 0 0.267 rpy=0 0 0 -> xyz=-0.001549459761 0.0003137374879 0.2656630874 rpy=-0.002122362144 -0.002407404361 2.55469422e-06
- joint joint2: origin xyz=0 0 0 rpy=-1.5708 0 0 -> xyz=0.0001424681977 -4.629010846e-07 -5.750245766e-11 rpy=-1.570928454 0.002410640009 -0.003248984925
- joint joint3: origin xyz=0.0535 -0.2845 0 rpy=0 0 0 -> xyz=0.05299152806 -0.2844330966 5.917066301e-05 rpy=-0.001330370083 -0.001908135135 -3.037097713e-06
- joint joint4: origin xyz=0.0775 0.3425 0 rpy=-1.5708 0 0 -> xyz=0.07818619162 0.3414653838 -0.0005268830573 rpy=-1.57233882 -0.001340431976 -0.002912688535
- joint joint5: origin xyz=0 0 0 rpy=1.5708 0 0 -> xyz=-0.0003658483038 -0.002068420639 -3.251171802e-05 rpy=1.586496472 -0.002846868243 -0.006097148173
- joint joint6: origin xyz=0.076 0.097 0 rpy=-1.5708 0 0 -> xyz=0.07646542042 0.0960168317 -0.0008099220577 rpy=-1.581605673 0.005988837685 -0.000228099816

File: rsc/robot/xarm_allegro.urdf (robot description, URDF)
Before this commit: robot combined_robot, 30 links, 29 joints
Joints:
- joint joint1: origin xyz=0 0 0.267 rpy=0 0 0 -> xyz=-0.001549459761 0.0003137374879 0.2656630874 rpy=-0.002122362144 -0.002407404361 2.55469422e-06
- joint joint2: origin xyz=0 0 0 rpy=-1.5708 0 0 -> xyz=0.0001424681977 -4.629010846e-07 -5.750245766e-11 rpy=-1.570928454 0.002410640009 -0.003248984925
- joint joint3: origin xyz=0.0535 -0.2845 0 rpy=0 0 0 -> xyz=0.05299152806 -0.2844330966 5.917066301e-05 rpy=-0.001330370083 -0.001908135135 -3.037097713e-06
- joint joint4: origin xyz=0.0775 0.3425 0 rpy=-1.5708 0 0 -> xyz=0.07818619162 0.3414653838 -0.0005268830573 rpy=-1.57233882 -0.001340431976 -0.002912688535
- joint joint5: origin xyz=0 0 0 rpy=1.5708 0 0 -> xyz=-0.0003658483038 -0.002068420639 -3.251171802e-05 rpy=1.586496472 -0.002846868243 -0.006097148173
- joint joint6: origin xyz=0.076 0.097 0 rpy=-1.5708 0 0 -> xyz=0.07646542042 0.0960168317 -0.0008099220577 rpy=-1.581605673 0.005988837685 -0.000228099816

File: rsc/robot/xarm_inspire_left.urdf (robot description, URDF)
Before this commit: robot combined_robot, 22 links, 21 joints
Links:
- removed link right_index_1
- removed link right_index_2
- removed link right_little_1
- removed link right_little_2
- removed link right_middle_1
- removed link right_middle_2
- removed link right_ring_1
- removed link right_ring_2
- removed link right_thumb_1
- removed link right_thumb_2
- removed link right_thumb_3
- removed link right_thumb_4
- added link left_index_1, mass 0.00719999389753264; collision mesh filename=inspire/meshes/left_index_1.STL; visual mesh filename=inspire/meshes/left_index_1.STL
- added link left_index_2, mass 0.0096859422185797; collision mesh filename=inspire/meshes/left_index_2.STL; visual mesh filename=inspire/meshes/left_index_2.STL
- added link left_little_1, mass 0.00719994987013217; collision mesh filename=inspire/meshes/left_little_1.STL; visual mesh filename=inspire/meshes/left_little_1.STL
- added link left_little_2, mass 0.0075928240732547; collision mesh filename=inspire/meshes/left_little_2.STL; visual mesh filename=inspire/meshes/left_little_2.STL
- added link left_middle_1, mass 0.00719999454699651; collision mesh filename=inspire/meshes/left_middle_1.STL; visual mesh filename=inspire/meshes/left_middle_1.STL
- added link left_middle_2, mass 0.0104603374357648; collision mesh filename=inspire/meshes/left_middle_2.STL; visual mesh filename=inspire/meshes/left_middle_2.STL
- added link left_ring_1, mass 0.00719998997814135; collision mesh filename=inspire/meshes/left_ring_1.STL; visual mesh filename=inspire/meshes/left_ring_1.STL
- added link left_ring_2, mass 0.0096859390369724; collision mesh filename=inspire/meshes/left_ring_2.STL; visual mesh filename=inspire/meshes/left_ring_2.STL
- added link left_thumb_1, mass 0.00115518743162309; collision mesh filename=inspire/meshes/left_thumb_1.STL; visual mesh filename=inspire/meshes/left_thumb_1.STL
- added link left_thumb_2, mass 0.016; collision mesh filename=inspire/meshes/left_thumb_2.STL; visual mesh filename=inspire/meshes/left_thumb_2.STL
- added link left_thumb_3, mass 0.012; collision mesh filename=inspire/meshes/left_thumb_3.STL; visual mesh filename=inspire/meshes/left_thumb_3.STL
- added link left_thumb_4, mass 0.01; collision mesh filename=inspire/meshes/left_thumb_4.STL; visual mesh filename=inspire/meshes/left_thumb_4.STL
- link base_link: geometry collision mesh filename=inspire/meshes/left_base_link.STL; visual mesh filename=inspire/meshes/left_base_link.STL
Joints:
- removed joint R_hand_base_joint
- removed joint right_index_1_joint
- removed joint right_index_2_joint
- removed joint right_little_1_joint
- removed joint right_little_2_joint
- removed joint right_middle_1_joint
- removed joint right_middle_2_joint
- removed joint right_ring_1_joint
- removed joint right_ring_2_joint
- removed joint right_thumb_1_joint
- removed joint right_thumb_2_joint
- removed joint right_thumb_3_joint
- removed joint right_thumb_4_joint
- added joint L_hand_base_joint: type fixed, parent wrist, child base_link, origin xyz=0 0 0 rpy=0 0 0
- added joint left_index_1_joint: type revolute, parent base_link, child left_index_1, origin xyz=0.038679 0.00056467 -0.1564 rpy=-1.5359 0 -1.5708, axis 0 0 1, limit lower=0 upper=1.6 effort=10 velocity=1
- added joint left_index_2_joint: type revolute, parent left_index_1, child left_index_2, origin xyz=-0.0016312 0.032734 -0.00055 rpy=0 0 0, axis 0 0 1, limit lower=0 upper=3.14 effort=10 velocity=1, mimic joint=left_index_1_joint multiplier=1.05 offset=0
- added joint left_little_1_joint: type revolute, parent base_link, child left_little_1, origin xyz=-0.025916 0.00056467 -0.15365 rpy=-1.6755 0 -1.5708, axis 0 0 1, limit lower=0 upper=1.6 effort=10 velocity=1
- added joint left_little_2_joint: type revolute, parent left_little_1, child left_little_2, origin xyz=-0.005182 0.032363 -0.00055 rpy=0 0 1.5708, axis 0 0 1, limit lower=0 upper=3.14 effort=10 velocity=1, mimic joint=left_little_1_joint multiplier=1.18 offset=0
- added joint left_middle_1_joint: type revolute, parent base_link, child left_middle_1, origin xyz=0.0171 0.00056467 -0.157 rpy=-1.5708 0 -1.5708, axis 0 0 1, limit lower=0 upper=1.6 effort=10 velocity=1
- added joint left_middle_2_joint: type revolute, parent left_middle_1, child left_middle_2, origin xyz=-0.0028436 0.032651 -0.00055 rpy=0 0 0, axis 0 0 1, limit lower=0 upper=3.14 effort=10 velocity=1, mimic joint=left_middle_1_joint multiplier=1.05 offset=0
- added joint left_ring_1_joint: type revolute, parent base_link, child left_ring_1, origin xyz=-0.0045302 0.00056467 -0.15683 rpy=-1.6232 0 -1.5708, axis 0 0 1, limit lower=0 upper=1.6 effort=10 velocity=1
- added joint left_ring_2_joint: type revolute, parent left_ring_1, child left_ring_2, origin xyz=-0.0031431 0.032624 -0.00055 rpy=0 0 0, axis 0 0 1, limit lower=0 upper=3.14 effort=10 velocity=1, mimic joint=left_ring_1_joint multiplier=1.05 offset=0
- added joint left_thumb_1_joint: type revolute, parent base_link, child left_thumb_1, origin xyz=0.0269 0.02101 -0.069 rpy=-3.1416 0 -3.1416, axis 0 0 -1, limit lower=0 upper=1.15 effort=10 velocity=1
- added joint left_thumb_2_joint: type revolute, parent left_thumb_1, child left_thumb_2, origin xyz=-0.0063016 0.011924 0.003 rpy=1.5708 0 2.7925, axis 0 0 1, limit lower=0 upper=0.55 effort=10 velocity=1
- added joint left_thumb_3_joint: type revolute, parent left_thumb_2, child left_thumb_3, origin xyz=0.034968 0.021325 -0.0015 rpy=0 0 0, axis 0 0 1, limit lower=0 upper=3.14 effort=10 velocity=1, mimic joint=left_thumb_2_joint multiplier=0.60 offset=0
- added joint left_thumb_4_joint: type revolute, parent left_thumb_3, child left_thumb_4, origin xyz=0.018887 0.011501 -0.0002 rpy=0 0 0, axis 0 0 1, limit lower=0 upper=3.14 effort=10 velocity=1, mimic joint=left_thumb_2_joint multiplier=0.8 offset=0
- joint arm_to_hand: origin xyz=0.00000 0.00000 0.0350 rpy=3.14159 0.00000 0.00000 -> xyz=0.00450 0 0.0350 rpy=3.14159 0.00000 0.00000
