Commit message: 0212_1321

File: rsc/robot/openarm/openarm_bimanual.urdf (robot description, URDF)
Before this commit: robot openarm, 26 links, 25 joints
Links:
- removed link openarm_left_hand
- removed link openarm_left_hand_tcp
- removed link openarm_left_left_finger
- removed link openarm_left_right_finger
- removed link openarm_right_hand
- removed link openarm_right_hand_tcp
- removed link openarm_right_left_finger
- removed link openarm_right_right_finger
Joints:
- removed joint left_openarm_hand_joint
- removed joint openarm_left_finger_joint1
- removed joint openarm_left_finger_joint2
- removed joint openarm_left_hand_tcp_joint
- removed joint openarm_right_finger_joint1
- removed joint openarm_right_finger_joint2
- removed joint openarm_right_hand_tcp_joint
- removed joint right_openarm_hand_joint
