Commit message: curobo

File: rsc/robot/xarm/xarm.urdf (robot description, URDF)
Before this commit: robot xarm6, 9 links, 8 joints
Links:
- removed link palm_link
- added link link_eef
- link link1: mass 2.16 -> 2.3814; geometry collision mesh filename=xarm_meshes/xarm6/visual/link1.stl; visual mesh filename=xarm_meshes/xarm6/visual/link1.stl
- link link2: mass 1.71 -> 2.2675; geometry collision mesh filename=xarm_meshes/xarm6/visual/link2.stl; visual mesh filename=xarm_meshes/xarm6/visual/link2.stl
- link link3: mass 1.384 -> 1.875; geometry collision mesh filename=xarm_meshes/xarm6/visual/link3.stl; visual mesh filename=xarm_meshes/xarm6/visual/link3.stl
- link link4: mass 1.115 -> 1.3192; geometry collision mesh filename=xarm_meshes/xarm6/visual/link4.stl; visual mesh filename=xarm_meshes/xarm6/visual/link4.stl
- link link5: mass 1.275 -> 1.33854; geometry collision mesh filename=xarm_meshes/xarm6/visual/link5.stl; visual mesh filename=xarm_meshes/xarm6/visual/link5.stl
- link link6: mass 0.1096 -> 0.17; geometry collision mesh filename=xarm_meshes/end_tool/collision/end_tool.stl; visual mesh filename=xarm_meshes/xarm6/visual/link6.stl
- link link_base: geometry collision mesh filename=xarm_meshes/xarm6/visual/link_base.stl; visual mesh filename=xarm_meshes/xarm6/visual/link_base.stl
Joints:
- removed joint gripper_base_joint
- added joint joint_eef: type fixed, parent link6, child link_eef, origin xyz=0 0 0 rpy=0 0 0
- joint joint1: limit lower=-6.28318530718 upper=6.28318530718 effort=500.0 velocity=3.14 -> lower=-6.283185307179586 upper=6.283185307179586 effort=50.0 velocity=3.14; origin xyz=0 0 0.267 rpy=0 0 0 -> xyz=-0.0010697057005017996 -0.0004954295000061393 0.2672901153564453 rpy=0.0029317450243979692 -0.0009082292672246695 -1.3313493809619104e-06
- joint joint2: origin xyz=0 0 0 rpy=-1.5708 0 0 -> xyz=0.0004169351886957884 1.990151190511824e-07 -9.557788588354654e-11 rpy=-1.569319725036621 0.0009085785131901503 0.00047865818487480283
- joint joint3: origin xyz=0.0535 -0.2845 0 rpy=0 0 0 -> xyz=0.05311902239918709 -0.28416889905929565 -0.0012295488268136978 rpy=0.0022015380673110485 0.0029121467377990484 -3.740997499335208e-06
- joint joint4: limit lower=-6.28318530718 upper=6.28318530718 effort=32.0 velocity=3.14 -> lower=-6.283185307179586 upper=6.283185307179586 effort=32.0 velocity=3.14; origin xyz=0.0775 0.3425 0 rpy=-1.5708 0 0 -> xyz=0.07675719261169434 0.34063249826431274 -0.0012138120364397764 rpy=-1.574359655380249 -0.0024353251792490482 -0.0006168704712763429
- joint joint5: limit lower=-1.69297 upper=3.14159265359 effort=32.0 velocity=3.14 -> lower=-1.69297 upper=3.141592653589793 effort=32.0 velocity=3.14; origin xyz=0 0 0 rpy=1.5708 0 0 -> xyz=-0.00036679222830571234 -0.0028716931119561195 -4.53642824140843e-05 rpy=1.5865709781646729 -0.0005549316992983222 -0.01099355798214674
- joint joint6: limit lower=-6.28318530718 upper=6.28318530718 effort=20.0 velocity=3.14 -> lower=-6.283185307179586 upper=6.283185307179586 effort=20.0 velocity=3.14; origin xyz=0.076 0.097 0 rpy=-1.5708 0 0 -> xyz=0.07698416709899902 0.09629102051258087 -0.001671688398346305 rpy=-1.5900110006332397 0.011010788381099701 -0.0004998284275643528
